Commit message: 成功实现第一条支链

File: test/3SPR.urdf (robot description, URDF)
Before this commit: robot 3SPR_Exact, 18 links, 17 joints
Links:
- removed link leg2_base_virtual
- removed link leg2_link1
- removed link leg2_link2
- removed link leg2_lower
- removed link leg2_tip
- removed link leg2_upper
- removed link leg3_base_virtual
- removed link leg3_link1
- removed link leg3_link2
- removed link leg3_lower
- removed link leg3_tip
- removed link leg3_upper
- removed link platform_link
- added link leg1_s_joint_end, mass 0.01
- link leg1_lower: geometry visual cylinder length=3.773502692 radius=0.1
- link leg1_upper: geometry visual cylinder length=2.0 radius=0.15
Joints:
- removed joint leg1_joint5
- removed joint leg2_base_fixed
- removed joint leg2_joint1
- removed joint leg2_joint2
- removed joint leg2_joint3
- removed joint leg2_joint4
- removed joint leg2_joint5
- removed joint leg3_base_fixed
- removed joint leg3_joint1
- removed joint leg3_joint2
- removed joint leg3_joint3
- removed joint leg3_joint4
- removed joint leg3_joint5
- added joint leg1_orientation_fix: type fixed, parent leg1_s_joint_end, child leg1_upper, origin xyz=0 0 0 rpy=0 0.523599 0
- joint leg1_joint1: origin xyz=3.886751346 0 0 rpy=0 0 0 -> xyz=3.887 0 0 rpy=0 0 0
- joint leg1_joint3: child leg1_upper -> leg1_s_joint_end
- joint leg1_joint4: axis -0.500000000 0 0.866025404 -> 0 0 -1; limit lower=0.0 upper=4.0 effort=5000 velocity=2.0 -> lower=-1 upper=2.0 effort=5000 velocity=2.0; origin xyz=0 0 0 rpy=0 0 0 -> xyz=0 0 -1 rpy=0 0 0

Commit message: feat: implement and verify first kinematic chain

File: test/3SPR.urdf (robot description, URDF)
Before this commit: robot 3SPR_Exact, 18 links, 17 joints
Links:
- removed link leg2_base_virtual
- removed link leg2_link1
- removed link leg2_link2
- removed link leg2_lower
- removed link leg2_tip
- removed link leg2_upper
- removed link leg3_base_virtual
- removed link leg3_link1
- removed link leg3_link2
- removed link leg3_lower
- removed link leg3_tip
- removed link leg3_upper
- removed link platform_link
- added link leg1_s_joint_end, mass 0.01
- added link motion_link, mass 1000.0; visual cylinder length=0.2 radius=1.5
- added link motion_upper, mass 20.0; visual cylinder length=0.5 radius=0.15
- link leg1_lower: geometry visual cylinder length=5.773502692 radius=0.1
- link leg1_upper: geometry visual cylinder length=0.5 radius=0.15
Joints:
- removed joint leg2_base_fixed
- removed joint leg2_joint1
- removed joint leg2_joint2
- removed joint leg2_joint3
- removed joint leg2_joint4
- removed joint leg2_joint5
- removed joint leg3_base_fixed
- removed joint leg3_joint1
- removed joint leg3_joint2
- removed joint leg3_joint3
- removed joint leg3_joint4
- removed joint leg3_joint5
- added joint leg1_motion_fix: type fixed, parent leg1_lower, child motion_upper, origin xyz=0 0 -5.773502692 rpy=1.570796 -0.523599 0
- added joint leg1_orientation_fix: type fixed, parent leg1_s_joint_end, child leg1_upper, origin xyz=0 0 0 rpy=0 0.523599 0
- joint leg1_joint1: origin xyz=3.886751346 0 0 rpy=0 0 0 -> xyz=3.887 0 0 rpy=0 0 0
- joint leg1_joint3: child leg1_upper -> leg1_s_joint_end
- joint leg1_joint4: axis -0.500000000 0 0.866025404 -> 0 0 -1; limit lower=0.0 upper=4.0 effort=5000 velocity=2.0 -> lower=-1 upper=2.0 effort=5000 velocity=2.0
- joint leg1_joint5: child platform_link -> motion_link; origin xyz=-2.886751346 0 5.000000000 rpy=0 0 0 -> xyz=0 0 0 rpy=0 0 0; parent leg1_lower -> motion_upper

Commit message: 完全实现第一条支链的模型，并且经过了check检验

File: test/3SPR.urdf (robot description, URDF)
Before this commit: robot Single_Leg_Open_Chain, 6 links, 5 joints
Links:
- added link motion_link, mass 1000.0; visual cylinder length=0.2 radius=1.5
- added link motion_upper, mass 20.0; visual cylinder length=0.5 radius=0.15
- link leg1_lower: geometry visual cylinder length=5.773502692 radius=0.1
- link leg1_upper: geometry visual cylinder length=0.5 radius=0.15
Joints:
- added joint leg1_joint5: type revolute, parent motion_upper, child motion_link, origin xyz=0 0 0 rpy=0 0 0, axis 0 1 0, limit lower=-1.57 upper=1.57 effort=0 velocity=0
- added joint leg1_motion_fix: type fixed, parent leg1_lower, child motion_upper, origin xyz=0 0 -5.773502692 rpy=1.570796 -0.523599 0
- joint leg1_joint4: origin xyz=0 0 -1 rpy=0 0 0 -> xyz=0 0 0 rpy=0 0 0
