Commit message: 完全对齐了坐标系、物体等内容，静态零位约束完全

File: test/real_3SPR.urdf (robot description, URDF)
Before this commit: robot 3_SPR_Parallel_Robot, 16 links, 15 joints
Links:
- removed link leg1_link1
- removed link leg1_link2
- removed link leg1_s_joint_end
- removed link leg2_link1
- removed link leg2_link2
- removed link leg2_s_joint_end
- removed link leg3_link1
- removed link leg3_link2
- removed link leg3_s_joint_end
- added link leg1_s1, mass 0.1
- added link leg1_s2, mass 0.1
- added link leg1_s3, mass 0.1
- added link leg2_anchor, mass 0.01
- added link leg2_s1, mass 0.1
- added link leg2_s2, mass 0.1
- added link leg2_s3, mass 0.1
- added link leg3_anchor, mass 0.01
- added link leg3_s1, mass 0.1
- added link leg3_s2, mass 0.1
- added link leg3_s3, mass 0.1
- link base_link: mass 1000.0 -> 100.0
- link leg1_lower: mass 15.0 -> 2.0; geometry visual cylinder length=7.7735 radius=0.1
- link leg2_lower: mass 15.0 -> 2.0; geometry visual cylinder length=7.7735 radius=0.1
- link leg3_lower: mass 15.0 -> 2.0; geometry visual cylinder length=7.7735 radius=0.1
- link motion_link: mass 50.0 -> 10.0; geometry visual cylinder length=0.2 radius=2
Joints:
- added joint leg2_anchor_joint: type fixed, parent motion_link, child leg2_anchor, origin xyz=-1.5 0.0 0.866025 rpy=0 -2.094395 0
- added joint leg3_anchor_joint: type fixed, parent motion_link, child leg3_anchor, origin xyz=-1.5 0.0 -0.866025  rpy=0.0 2.094395 0.0
- joint leg1_joint1: axis 0.866025 0 -0.5 -> 0.866025 0.0 -0.5; child leg1_link1 -> leg1_s1; limit lower=-1.57 upper=1.57 effort=100 velocity=1 -> lower=-1.57 upper=1.57 effort=100.0 velocity=1.0; origin xyz=3.887 0 0 rpy=0 0 0 -> xyz=3.88675 0.0 0.0 rpy=0.0 0.0 0.0
- joint leg1_joint2: axis 0 1 0 -> 0.0 1.0 0.0; child leg1_link2 -> leg1_s2; limit lower=-1.57 upper=1.57 effort=100 velocity=1 -> lower=-1.57 upper=1.57 effort=100.0 velocity=1.0; origin (none) -> xyz=0.0 0.0 0.0 rpy=0.0 0.0 0.0; parent leg1_link1 -> leg1_s1
- joint leg1_joint3: axis -0.5 0 -0.866025 -> -0.5 0.0 -0.866025; child leg1_s_joint_end -> leg1_s3; limit lower=-1.57 upper=1.57 effort=100 velocity=1 -> lower=-1.57 upper=1.57 effort=100.0 velocity=1.0; origin (none) -> xyz=0.0 0.0 0.0 rpy=0.0 0.0 0.0; parent leg1_link2 -> leg1_s2
- joint leg1_joint4: axis 0 0 -1 -> 0.0 0.0 -1.0; limit lower=-1 upper=2.0 effort=5000 velocity=2.0 -> lower=1.0 upper=-2.0 effort=5000.0 velocity=2.0; origin xyz=0 0 0 rpy=0 0.523599 0 -> xyz=0.0 0.0 0.0 rpy=0.0 0.523599 0.0; parent leg1_s_joint_end -> leg1_s3
- joint leg1_joint5: axis 0 1 0 -> 0.0 1.0 0.0; limit lower=-1.57 upper=1.57 effort=100 velocity=1 -> lower=-1.57 upper=1.57 effort=100.0 velocity=1.0; origin xyz=0 0 -5.7735 rpy=1.570796 -0.523599 0 -> xyz=0.0 0.0 -5.7735 rpy=1.570796 -0.523599 0.0
- joint leg2_joint1: axis 0.866025 0 -0.5 -> 0.866025 0.0 -0.5; child leg2_link1 -> leg2_s1; limit lower=-1.57 upper=1.57 effort=100 velocity=1 -> lower=-1.57 upper=1.57 effort=100.0 velocity=1.0; origin xyz=-1.9435 3.3662 0 rpy=0 0 2.0944 -> xyz=-1.943376 3.366025 0.0 rpy=0.0 0.0 2.094395
- joint leg2_joint2: axis 0 1 0 -> 0.0 1.0 0.0; child leg2_link2 -> leg2_s2; limit lower=-1.57 upper=1.57 effort=100 velocity=1 -> lower=-1.57 upper=1.57 effort=100.0 velocity=1.0; origin (none) -> xyz=0.0 0.0 0.0 rpy=0.0 0.0 0.0; parent leg2_link1 -> leg2_s1
- joint leg2_joint3: axis -0.5 0 -0.866025 -> -0.5 0.0 -0.866025; child leg2_s_joint_end -> leg2_s3; limit lower=-1.57 upper=1.57 effort=100 velocity=1 -> lower=-1.57 upper=1.57 effort=100.0 velocity=1.0; origin (none) -> xyz=0.0 0.0 0.0 rpy=0.0 0.0 0.0; parent leg2_link2 -> leg2_s2
- joint leg2_joint4: axis 0 0 -1 -> 0.0 0.0 -1.0; limit lower=-1 upper=2.0 effort=5000 velocity=2.0 -> lower=1.0 upper=-2.0 effort=5000.0 velocity=2.0; origin xyz=0 0 0 rpy=0 0.523599 0 -> xyz=0.0 0.0 0.0 rpy=0.0 0.523599 0.0; parent leg2_s_joint_end -> leg2_s3
- joint leg2_joint5: axis 0 1 0 -> 0.0 1.0 0.0; limit lower=-1.57 upper=1.57 effort=100 velocity=1 -> lower=-1.57 upper=1.57 effort=100.0 velocity=1.0; origin xyz=0 0 -5.7735 rpy=1.570796 -0.523599 0 -> xyz=0.0 0.0 -5.7735 rpy=1.570796 -0.523599 0.0
- joint leg3_joint1: axis 0.866025 0 -0.5 -> 0.866025 0.0 -0.5; child leg3_link1 -> leg3_s1; limit lower=-1.57 upper=1.57 effort=100 velocity=1 -> lower=-1.57 upper=1.57 effort=100.0 velocity=1.0; origin xyz=-1.9435 -3.3662 0 rpy=0 0 4.1888 -> xyz=-1.943376 -3.366025 0.0 rpy=0.0 0.0 -2.094395
- joint leg3_joint2: axis 0 1 0 -> 0.0 1.0 0.0; child leg3_link2 -> leg3_s2; limit lower=-1.57 upper=1.57 effort=100 velocity=1 -> lower=-1.57 upper=1.57 effort=100.0 velocity=1.0; origin (none) -> xyz=0.0 0.0 0.0 rpy=0.0 0.0 0.0; parent leg3_link1 -> leg3_s1
- joint leg3_joint3: axis -0.5 0 -0.866025 -> -0.5 0.0 -0.866025; child leg3_s_joint_end -> leg3_s3; limit lower=-1.57 upper=1.57 effort=100 velocity=1 -> lower=-1.57 upper=1.57 effort=100.0 velocity=1.0; origin (none) -> xyz=0.0 0.0 0.0 rpy=0.0 0.0 0.0; parent leg3_link2 -> leg3_s2
- joint leg3_joint4: axis 0 0 -1 -> 0.0 0.0 -1.0; limit lower=-1 upper=2.0 effort=5000 velocity=2.0 -> lower=1.0 upper=-2.0 effort=5000.0 velocity=2.0; origin xyz=0 0 0 rpy=0 0.523599 0 -> xyz=0.0 0.0 0.0 rpy=0.0 0.523599 0.0; parent leg3_s_joint_end -> leg3_s3
- joint leg3_joint5: axis 0 1 0 -> 0.0 1.0 0.0; limit lower=-1.57 upper=1.57 effort=100 velocity=1 -> lower=-1.57 upper=1.57 effort=100.0 velocity=1.0; origin xyz=0 0 -5.7735 rpy=1.570796 -0.523599 0 -> xyz=0.0 0.0 -5.7735 rpy=1.570796 -0.523599 0.0
