Commit message: 完全闭合了CloseLoop,闭环误差err均为0

File: test/real_3SPR_copy.urdf (robot description, URDF)
Before this commit: robot 3SPR_Parallel_Robot, 18 links, 17 joints
Links:
- removed link leg2_anchor
- removed link leg2_tip
- removed link leg3_anchor
- removed link leg3_tip
- added link leg2_anchor_frame, mass 0.001
- added link leg2_tip_frame, mass 0.01
- added link leg3_anchor_frame, mass 0.001
- added link leg3_tip_frame, mass 0.01
- link motion_link: geometry visual cylinder length=0.2 radius=1.5
Joints:
- joint leg1_joint2: origin xyz=0.0 0.0 0.0 rpy=0.0 0.0 0.0 -> (none)
- joint leg1_joint3: origin xyz=0.0 0.0 0.0 rpy=0.0 0.0 0.0 -> (none)
- joint leg2_anchor_joint: child leg2_anchor -> leg2_anchor_frame; origin xyz=-1.5 0.0 0.866025 rpy=0 -2.094395 0 -> xyz=-1.5 0 -0.866025 rpy=0 -2.094395 0
- joint leg2_joint2: origin xyz=0.0 0.0 0.0 rpy=0.0 0.0 0.0 -> (none)
- joint leg2_joint3: origin xyz=0.0 0.0 0.0 rpy=0.0 0.0 0.0 -> (none)
- joint leg2_joint5: child leg2_tip -> leg2_tip_frame
- joint leg3_anchor_joint: child leg3_anchor -> leg3_anchor_frame; origin xyz=-1.5 0.0 -0.866025  rpy=0.0 2.094395 0.0 -> xyz=-1.5 0 0.866025  rpy=0.0 2.094395 0.0
- joint leg3_joint2: origin xyz=0.0 0.0 0.0 rpy=0.0 0.0 0.0 -> (none)
- joint leg3_joint3: origin xyz=0.0 0.0 0.0 rpy=0.0 0.0 0.0 -> (none)
- joint leg3_joint5: child leg3_tip -> leg3_tip_frame

Commit message: rpy固定角绕z旋转了120°，以测试消除雅可比矩阵某行的巨大数值

File: test/real_3SPR_copy.urdf (robot description, URDF)
Before this commit: robot 3SPR_Parallel_Robot, 18 links, 17 joints
Joints:
- joint leg2_joint5: origin xyz=0.0 0.0 -5.7735 rpy=1.570796 -0.523599 0.0 -> xyz=0.0 0.0 -5.7735 rpy=1.570796 -0.523599 2.094395
- joint leg3_joint5: origin xyz=0.0 0.0 -5.7735 rpy=1.570796 -0.523599 0.0 -> xyz=0.0 0.0 -5.7735 rpy=1.570796 -0.523599 0
